Commit message: 新文件：   .vscode/c_cpp_properties.json 	新文件：   .vscode/settings.json 	修改：     turtlebot3_description/urdf/turtlebot3_burger.gazebo.xacro 	修改：     turtlebot3_description/urdf/turtlebot3_burger.urdf.xacro 	修改：     turtlebot3_description/urdf/turtlebot3_waffle_pi.urdf.xacro 	新文件：   turtlebot3_description/urdf/turtlebot3_waffle_pive.gazebo.xacro 	新文件：   turtlebot3_description/urdf/turtlebot3_waffle_pive.urdf.xacro

File: turtlebot3_description/urdf/turtlebot3_burger.urdf.xacro (robot description, xacro)
@@ -3,4 +3,12 @@
   <xacro:include filename="$(find turtlebot3_description)/urdf/common_properties.xacro"/>
   <xacro:include filename="$(find turtlebot3_description)/urdf/turtlebot3_burger.gazebo.xacro"/>
+  <!-- VLP-16 -->
+  <xacro:include filename="$(find velodyne_description)/urdf/VLP-16.urdf.xacro"/>
+  <VLP-16 parent="base_link" name="velodyne" topic="velodyne_points" hz="10" samples="1024" gpu="true" lasers="16" max_range="100">
+    <origin xyz="-0.032 0.0 0.15" rpy="0 0 0" />
+  </VLP-16>
+    <!-- <xacro:vlp16_mount prefix="" parent_link="base_link" topic="velodyne_points">
+      <origin xyz="-0.032 0 0.173" rpy="0 0 0" />
+    </xacro:vlp16_mount> -->
   <link name="base_footprint"/>
   <joint name="base_joint" type="fixed">
@@ -113,10 +121,10 @@
   </joint>
   <link name="imu_link"/>
-  <joint name="scan_joint" type="fixed">
+  <!-- <joint name="scan_joint" type="fixed">
     <parent link="base_link"/>
     <child link="base_scan"/>
     <origin xyz="-0.032 0 0.172" rpy="0 0 0"/>
-  </joint>
-  <link name="base_scan">
+  </joint> -->
+  <!-- <link name="base_scan">
     <visual>
       <origin xyz="0 0 0.0" rpy="0 0 0"/>
@@ -139,4 +147,4 @@
                izz="0.001" />
     </inertial>
-  </link>
+  </link> -->
 </robot>

File: turtlebot3_description/urdf/turtlebot3_waffle_pive.gazebo.xacro (robot description, xacro)
@@ -1,6 +1,7 @@
 <?xml version="1.0"?>
-<robot name="turtlebot3_burger_sim" xmlns:xacro="http://ros.org/wiki/xacro">
-  <xacro:arg name="laser_visual" default="false"/>
-  <xacro:arg name="imu_visual"   default="false"/>
+<robot name="turtlebot3_waffle_pi_sim" xmlns:xacro="http://ros.org/wiki/xacro">
+  <xacro:arg name="laser_visual"  default="false"/>
+  <xacro:arg name="camera_visual" default="false"/>
+  <xacro:arg name="imu_visual"    default="false"/>
   <gazebo reference="base_link">
     <material>Gazebo/DarkGrey</material>
@@ -26,5 +27,14 @@
     <material>Gazebo/FlatBlack</material>
   </gazebo>
-  <gazebo reference="caster_back_link">
+  <gazebo reference="caster_back_right_link">
+    <mu1>0.1</mu1>
+    <mu2>0.1</mu2>
+    <kp>1000000.0</kp>
+    <kd>100.0</kd>
+    <minDepth>0.001</minDepth>
+    <maxVel>1.0</maxVel>
+    <material>Gazebo/FlatBlack</material>
+  </gazebo>
+  <gazebo reference="caster_back_left_link">
     <mu1>0.1</mu1>
     <mu2>0.1</mu2>
@@ -40,8 +50,8 @@
       <visualize>$(arg imu_visual)</visualize>
     </sensor>
-    <material>Gazebo/FlatBlack</material>
+    <material>Gazebo/Grey</material>
   </gazebo>
   <gazebo>
-    <plugin name="turtlebot3_burger_controller" filename="libgazebo_ros_diff_drive.so">
+    <plugin name="turtlebot3_waffle_pi_controller" filename="libgazebo_ros_diff_drive.so">
       <commandTopic>cmd_vel</commandTopic>
       <odometryTopic>odom</odometryTopic>
@@ -57,5 +67,5 @@
       <leftJoint>wheel_left_joint</leftJoint>
       <rightJoint>wheel_right_joint</rightJoint>
-      <wheelSeparation>0.160</wheelSeparation>
+      <wheelSeparation>0.287</wheelSeparation>
       <wheelDiameter>0.066</wheelDiameter>
       <wheelAcceleration>1</wheelAcceleration>
@@ -92,5 +102,5 @@
     </plugin>
   </gazebo>
-  <!-- <gazebo reference="base_scan">
+  <gazebo reference="base_scan">
     <material>Gazebo/FlatBlack</material>
     <sensor type="ray" name="lds_lfcd_sensor">
@@ -123,39 +133,37 @@
       </plugin>
     </sensor>
-  </gazebo> -->
-    <gazebo>
-    <!-- <plugin name="mecanum_controller" filename="libgazebo_ros_planar_move.so">
-        <commandTopic>cmd_vel</commandTopic>
-        <odometryTopic>odom</odometryTopic>
-        <odometryFrame>odom</odometryFrame>
-        <leftFrontJoint>front_left_wheel</leftFrontJoint>
-        <rightFrontJoint>front_right_wheel</rightFrontJoint>
-        <leftRearJoint>rear_left_wheel</leftRearJoint>
-        <rightRearJoint>rear_right_wheel</rightRearJoint>
-        <odometryRate>20.0</odometryRate>
-        <robotBaseFrame>base_link</robotBaseFrame> -->
-        <!-- </plugin>
-        <plugin name="p3d_base_controller" filename="libgazebo_ros_p3d.so">
+  </gazebo>
+<!--link : https://www.raspberrypi.org/documentation/hardware/camera/-->
+  <gazebo reference="camera_rgb_frame">
+    <sensor type="camera" name="Pi Camera">
+      <always_on>true</always_on>
+      <visualize>$(arg camera_visual)</visualize>
+      <camera>
+          <horizontal_fov>1.085595</horizontal_fov>
+          <image>
+              <width>640</width>
+              <height>480</height>
+              <format>R8G8B8</format>
+          </image>
+          <clip>
+              <near>0.03</near>
+              <far>100</far>
+          </clip>
+      </camera>
+      <plugin name="camera_controller" filename="libgazebo_ros_camera.so">
         <alwaysOn>true</alwaysOn>
-        <updateRate>50.0</updateRate>
-        <bodyName>base_link</bodyName>
-        <topicName>ground_truth/state</topicName>
-        <gaussianNoise>0.01</gaussianNoise>
-        <frameName>world</frameName>
-        <xyzOffsets>0 0 0</xyzOffsets>
-        <rpyOffsets>0 0 0</rpyOffsets>
-        </plugin> -->
-    </gazebo>
-    <!-- <gazebo>
-			<plugin name="p3d_base_controller" filename="libgazebo_ros_p3d.so">
-    		<alwaysOn>true</alwaysOn>
-    		<updateRate>50.0</updateRate>
-    		<bodyName>base_footprint</bodyName>
-   			<topicName>ground_truth/state</topicName>
-    		<gaussianNoise>0.01</gaussianNoise>
-    		<frameName>world</frameName>
-    		<xyzOffsets>0 0 0</xyzOffsets>
-   			<rpyOffsets>0 0 0</rpyOffsets>
- 			</plugin>
-		</gazebo> -->
+        <updateRate>30.0</updateRate>
+        <cameraName>camera</cameraName>
+        <frameName>camera_rgb_optical_frame</frameName>
+        <imageTopicName>rgb/image_raw</imageTopicName>
+        <cameraInfoTopicName>rgb/camera_info</cameraInfoTopicName>
+        <hackBaseline>0.07</hackBaseline>
+        <distortionK1>0.0</distortionK1>
+        <distortionK2>0.0</distortionK2>
+        <distortionK3>0.0</distortionK3>
+        <distortionT1>0.0</distortionT1>
+        <distortionT2>0.0</distortionT2>
+      </plugin>
+    </sensor>
+  </gazebo>
 </robot>

File: turtlebot3_description/urdf/turtlebot3_waffle_pive.urdf.xacro (robot description, xacro)
@@ -4,4 +4,8 @@
   <xacro:include filename="$(find turtlebot3_description)/urdf/turtlebot3_waffle_pi.gazebo.xacro"/>
   <link name="base_footprint"/>
+  <xacro:include filename="$(find velodyne_description)/urdf/VLP-16.urdf.xacro"/>
+  <VLP-16 parent="base_link" name="velodyne" topic="velodyne_points" hz="10" samples="1024" gpu="true" lasers="16" max_range="15">
+        <origin xyz="-0.064 0.0 0.50" rpy="0 0 0" />
+  </VLP-16>
   <joint name="base_joint" type="fixed">
     <parent link="base_footprint"/>
